File: Hardware/Rev1/Keyboard.sch (KiCad schematic (older format))
At the start: 41 parts

Commit message: Annotate Schematic
Parts:
- gave numbers to parts that had none: 41

Commit message: Change RGB-LED Symbols and assign PCB Footprints
Parts:
- BT1, BT2: footprint (none) -> guri-lib:BH-311P-1
- C1, C10, C2, C4, C5, C6, C7, C8, C9: footprint (none) -> Capacitors_SMD:C_0603
- C3: footprint (none) -> Capacitors_SMD:C_0805
- D1, D2: footprint (none) -> Diodes_SMD:SOD-123
- D3: footprint (none) -> guri-lib:OSTB0603C1C-A; symbol LED_RABG -> LED_ARBG
- D4: footprint (none) -> LEDs:LED-0603
- P1: footprint (none) -> guri-lib:ZX62R-B-5P
- Q1, Q2, Q3, Q4: footprint (none) -> TO_SOT_Packages_SMD:SOT-23
- R1, R10, R11, R12, R13, R14, R15, R2, R3, R4, R5, R6, R7, R8, R9: footprint (none) -> Resistors_SMD:R_0603
- SW1: value SW_PUSH -> ISP; footprint (none) -> guri-lib:SKRPACE010
- U1: footprint (none) -> Housings_DFN_QFN:QFN-32-1EP_5x5mm_Pitch0.5mm
- U2: footprint (none) -> guri-lib:SOT-223
- U3: footprint (none) -> guri-lib:HRM1026
- X1: footprint (none) -> Crystals:crystal_FA238-TSX3225

Commit message: Fix schematic
Connections:
- net labels removed: USB_Detect
Other:
- moved on the sheet: C4
Changed lines of the file:
@@
 L C C4
 U 1 1 5A49C99D
-P 2750 2800
-F 0 "C4" H 2775 2900 50  0000 L CNN
-F 1 "0.1u" H 2775 2700 50  0000 L CNN
-F 2 "Capacitors_SMD:C_0603" H 2788 2650 50  0001 C CNN
-F 3 "" H 2750 2800 50  0000 C CNN
-	1    2750 2800
+P 6550 2200
+F 0 "C4" H 6575 2300 50  0000 L CNN
+F 1 "0.1u" H 6575 2100 50  0000 L CNN
+F 2 "Capacitors_SMD:C_0603" H 6588 2050 50  0001 C CNN
+F 3 "" H 6550 2200 50  0000 C CNN
+	1    6550 2200
 	1    0    0    -1
 $EndComp
@@
 	3000 2900 3100 2900
 Wire Wire Line
-	2750 2650 2750 2600
-Connection ~ 2750 2600
-Wire Wire Line
-	2750 2950 2750 3000
-Connection ~ 2750 3000
-Wire Wire Line
 	2400 2650 2400 2600
 Connection ~ 2400 2600
@@
 	2000 7300 2000 7200
 Wire Wire Line
-	6800 2400 6850 2400
+	6550 2400 6850 2400
 Wire Wire Line
 	6800 2200 6800 2450
 Wire Wire Line
-	6850 2000 6800 2000
+	6550 2000 6850 2000
 Wire Wire Line
 	6800 2000 6800 1950
@@
 	7150 6350 7250 6350
 Text GLabel 7250 6350 2    60   Output ~ 0
-USB_Detect
+USBDetect
+Wire Wire Line
+	6550 2000 6550 2050
+Connection ~ 6800 2000
+Wire Wire Line
+	6550 2400 6550 2350
 $EndSCHEMATC

Commit message: Add Rev1 Left PCB Pattern
Parts:
- BT1, BT2: symbol Battery -> Battery_Cell
- U2: symbol AP1117D33 -> AP1117-33
- X1: footprint Crystals:crystal_FA238-TSX3225 -> Crystals:Crystal_SMD_3225-4pin_3.2x2.5mm; symbol CRYSTAL_SMD -> Crystal_GND24
Connections:
- net labels added: Col.1, Col.2, Col.3, Col.4, Col.5, Col.6, Col.7, Col.8, RowA, RowB, RowC, RowD
- net labels removed: Col.A, Col.B, Col.C, Col.D, Row1, Row2, Row3, Row4, Row5, Row6, Row7, Row8
- wire segments 145 -> 153
- no-connect marks 0 -> 11
Other:
- moved on the sheet: C10, C2, C6, C7, C8, C9, Q3, R13, R14, R4, U2
