File: Hardware/Rev1/SwitchAndLEDs.sch (KiCad schematic (older format))
At the start: 88 parts

Commit message: Annotate Schematic
Parts:
- gave numbers to parts that had none: 88

Commit message: Change RGB-LED Symbols and assign PCB Footprints
Parts:
- D10, D11, D12, D13, D14, D15, D16, D17, D18, D19, D20, D21, D22, D23, D24, D25, D26, D27, D28, D29, D30, D31, D32, D33, D34, D35, D36, D37, D38, D39, D9: footprint (none) -> Diodes_ThroughHole:Diode_DO-35_SOD27_Horizontal_RM10
- D5, D6, D7, D8: footprint (none) -> guri-lib:OSTB0603C1C-A; symbol LED_RABG -> LED_ARBG
- Q10, Q11, Q12, Q13, Q14, Q15, Q5, Q6, Q7, Q8, Q9: footprint (none) -> TO_SOT_Packages_SMD:SOT-23
- R16, R17, R18, R19, R20, R21, R22, R23, R24, R25, R26: footprint (none) -> Resistors_SMD:R_0603
- SW10, SW11, SW12, SW13, SW14, SW15, SW16, SW17, SW18, SW19, SW2, SW20, SW21, SW22, SW23, SW24, SW25, SW26, SW27, SW28, SW29, SW3, SW30, SW31, SW32, SW4, SW5, SW6, SW7, SW8, SW9: footprint (none) -> guri-lib:MX_PCB_Mount
Connections:
- net at Q7.3 (D): now also D5.1 (COMMON_ANODE); no longer D5.2 (COMMON_ANODE)
- net at D6.2 (RED_CATHODE): now also D5.2 (RED_CATHODE), D7.2 (RED_CATHODE), D8.2 (RED_CATHODE), R18.1; no longer Q8.3 (D)
- net at Q9.3 (D): now also D7.1 (COMMON_ANODE); no longer D7.2 (COMMON_ANODE)
- net at Q10.3 (D): now also D8.1 (COMMON_ANODE); no longer D8.2 (COMMON_ANODE)
- new net: D6.1 (COMMON_ANODE), Q8.3 (D)

Commit message: Add Rev1 Left PCB Pattern
Parts:
- D10, D11, D12, D13, D14, D15, D16, D17, D18, D19, D20, D21, D22, D23, D24, D25, D26, D27, D28, D29, D30, D31, D32, D33, D34, D35, D36, D37, D38, D39, D9: footprint Diodes_ThroughHole:Diode_DO-35_SOD27_Horizontal_RM10 -> Diodes_SMD:D_SOD-123
Connections:
- net Col.A renamed RowA
- net Col.B renamed RowB
- net Col.C renamed RowC
- net Col.D renamed RowD
- net Row1 renamed Col.1
- net Row2 renamed Col.2
- net Row3 renamed Col.3
- net Row4 renamed Col.4
- net Row5 renamed Col.5
- net Row6 renamed Col.6
- net Row7 renamed Col.7
- net Row8 renamed Col.8
